File: Cosmonode_ext06/Cosmonode_ext06.sch (KiCad schematic (older format))
At the start: 37 parts, among them J3 CONN_01X08, J4 CONN_01X08, J5 GS3, U1 XC6206P502MR

Commit message: big push2
Parts:
- removed C?: 100nF, symbol C
- removed J5, J?: GS3, Connectors:GS3, symbol GS3
- removed R? (x3): 100k, symbol R
- removed R? (x2): 33k, symbol R
- removed U1: XC6206P502MR, TO_SOT_Packages_SMD:SOT-23_Handsoldering, symbol PMIC-LDO-XC6206P302MR(SOT23)
- removed U?: TL082, symbol TL082
- added J2: Aloes_Logo, Aloes:Aloes_mini, symbol CONN_01X01
- added J3: OSHW_Logo, Symbols:OSHW-Logo_5.7x6mm_SilkScreen, symbol CONN_01X01
- C1, C10, C11, C12, C2, C3, C4, C5, C6, C7, C8, C9: renamed from C?; footprint (none) -> Capacitors_SMD:C_0603_HandSoldering
- D1: renamed from D?; footprint (none) -> LEDs:LED_0603_HandSoldering
- J1: renamed from J?; footprint TE_227161-1 -> BNC_P7003:TE_227161-1
- J4: renamed from J3; footprint Pin_Headers:Pin_Header_Straight_1x08_Pitch2.54mm -> Socket_Strips:Socket_Strip_Straight_1x08_Pitch2.54mm
- J6: renamed from J4; footprint Pin_Headers:Pin_Header_Straight_1x08_Pitch2.54mm -> Socket_Strips:Socket_Strip_Straight_1x08_Pitch2.54mm
- R1: renamed from 4,7M; value R -> 4,7M; footprint (none) -> Resistors_SMD:R_0603_HandSoldering
- R2, R3, R4, R5, R6, R8: renamed from R?; footprint (none) -> Resistors_SMD:R_0603_HandSoldering
- RV1: renamed from RV?; footprint (none) -> Potentiometers:Potentiometer_Trimmer_Bourns_3296W
- U1, U2, U3: renamed from U?; footprint SOIC127P600X175-8N -> Housings_SOIC:SOIC-8_3.9x4.9mm_Pitch1.27mm
Connections:
- net +5V is gone; now on net +3V3: C10.1, C2.2, C4.1, C8.1, R8.2, U1.7 (V+), U2.6 (LV), U2.8 (V+)
- net A1: now also R6.2, U3.6 (OUT)
- net -5V renamed -3V3
- net A_REF renamed A7
- no-connect marks 13 -> 21
