File: Cosmonode_ext01/Cosmonode_ext_01.sch (KiCad schematic (older format))
At the start: 15 parts, among them J1 GS2, J2 GS3, J3 CONN_01X07, J5 CONN_01X07, J7 GS3, J8 GS3, J9 GS3, U1 TSL2561T(6P-3.8X2.6MM), U2 BMP180, U3 SI7020-A20-YM0R

Commit message: fully update to v0.3
Parts:
- removed J2, J7: GS3, Connectors:GS3, symbol GS3
- added J4: Aloes_Logo, Aloes:Aloes_mini, symbol CONN_01X01
- added J6: OSHW_Logo, Symbols:OSHW-Logo_5.7x6mm_SilkScreen, symbol CONN_01X01
- J3, J5: value CONN_01X07 -> CONN_01X08; footprint Pin_Headers:Pin_Header_Straight_1x07_Pitch2.54mm -> Socket_Strips:Socket_Strip_Straight_1x08_Pitch2.54mm; symbol CONN_01X07 -> CONN_01X08
- U1: footprint TSL2561T_6P-3.8X2.6MM_:TMB6-1.55-3.8X2.6MM -> TSL2561T:TMB6-1.55-3.8X2.6MM
Connections:
- net at C1.1, J1.1 (G1), U1.1 (VDD): now also C2.1, C3.1, C4.1, J9.2 (G2), U2.2 (VDD), U2.3 (VDDIO), U3.5 (VDD)
- new net A6: J3.8 (P8)
- new net A7: J5.8 (P8)
- no-connect marks 6 -> 12
Other:
- note removed: "D5 as +3.3V"
- note removed: "D7 as +3.3V"
- moved on the sheet: J9
Changed lines of the file:
@@
 LIBS:BMP180
 LIBS:SI7020-A20-YM0R
-LIBS:TSL2561T_6P-3.8X2.6MM_
 LIBS:Cosmonode_ext_01-cache
 EELAYER 25 0
@@
 $EndDescr
 $Comp
-L CONN_01X07 J3
+L CONN_01X08 J3
 U 1 1 598047BC
-P 3750 4000
-F 0 "J3" H 3750 4400 50  0000 C CNN
-F 1 "CONN_01X07" V 3850 4000 50  0000 C CNN
-F 2 "Pin_Headers:Pin_Header_Straight_1x07_Pitch2.54mm" H 3750 4000 50  0001 C CNN
-F 3 "" H 3750 4000 50  0001 C CNN
-	1    3750 4000
-	1    0    0    -1
-$EndComp
-$Comp
-L CONN_01X07 J5
+P 3750 4050
+F 0 "J3" H 3750 4450 50  0000 C CNN
+F 1 "CONN_01X08" V 3850 4050 50  0000 C CNN
+F 2 "Socket_Strips:Socket_Strip_Straight_1x08_Pitch2.54mm" H 3750 4050 50  0001 C CNN
+F 3 "" H 3750 4050 50  0001 C CNN
+	1    3750 4050
+	1    0    0    -1
+$EndComp
+$Comp
+L CONN_01X08 J5
 U 1 1 598047EF
-P 4700 4000
-F 0 "J5" H 4700 4400 50  0000 C CNN
-F 1 "CONN_01X07" V 4800 4000 50  0000 C CNN
-F 2 "Pin_Headers:Pin_Header_Straight_1x07_Pitch2.54mm" H 4700 4000 50  0001 C CNN
-F 3 "" H 4700 4000 50  0001 C CNN
-	1    4700 4000
+P 4700 4050
+F 0 "J5" H 4700 4450 50  0000 C CNN
+F 1 "CONN_01X08" V 4800 4050 50  0000 C CNN
+F 2 "Socket_Strips:Socket_Strip_Straight_1x08_Pitch2.54mm" H 4700 4050 50  0001 C CNN
+F 3 "" H 4700 4050 50  0001 C CNN
+	1    4700 4050
 	1    0    0    -1
 $EndComp
@@
 F 0 "U1" H 4100 2650 50  0000 L BNN
 F 1 "TSL2561T(6P-3.8X2.6MM)" H 4350 2650 50  0000 L BNN
-F 2 "TSL2561T_6P-3.8X2.6MM_:TMB6-1.55-3.8X2.6MM" H 4350 2450 50  0001 L BNN
+F 2 "TSL2561T:TMB6-1.55-3.8X2.6MM" H 4350 2450 50  0001 L BNN
 F 3 "TSL2561T" H 4350 2450 50  0001 L BNN
 F 4 "2.50 USD" H 4350 2450 50  0001 L BNN "Price"
@@
 	1    0    0    -1
 $EndComp
-Text Label 3550 1650 2    60   ~ 0
-D5
 Text Label 5400 3400 0    60   ~ 0
 D6
@@
 Text Label 4750 2450 0    60   ~ 0
 D3
-Text Notes 3350 1650 2    60   ~ 0
-D5 as +3.3V
 Text Notes 5800 3500 2    60   ~ 0
 D6 as GND
-Text Notes 6950 1800 2    60   ~ 0
+Text Notes 7500 1500 2    60   ~ 0
 D4 as +3.3V
 NoConn ~ 5750 2550
@@
 Text Label 5750 2350 2    60   ~ 0
 A5
-Text Label 6800 3400 2    60   ~ 0
-D7
-$Comp
-L GS3 J2
-U 1 1 59805661
-P 3650 1800
-F 0 "J2" H 3700 2000 50  0000 C CNN
-F 1 "GS3" H 3700 1601 50  0000 C CNN
-F 2 "Connectors:GS3" V 3738 1726 50  0001 C CNN
-F 3 "" H 3650 1800 50  0001 C CNN
-	1    3650 1800
-	0    1    1    0
-$EndComp
 $Comp
 L GS3 J9
 U 1 1 5980583B
-P 7250 1950
-F 0 "J9" H 7300 2150 50  0000 C CNN
-F 1 "GS3" H 7300 1751 50  0000 C CNN
-F 2 "Connectors:GS3" V 7338 1876 50  0001 C CNN
-F 3 "" H 7250 1950 50  0001 C CNN
-	1    7250 1950
+P 7850 1700
+F 0 "J9" H 7900 1900 50  0000 C CNN
+F 1 "GS3" H 7900 1501 50  0000 C CNN
+F 2 "Connectors:GS3" V 7938 1626 50  0001 C CNN
+F 3 "" H 7850 1700 50  0001 C CNN
+	1    7850 1700
 	0    1    1    0
 $EndComp
-$Comp
-L GS3 J7
-U 1 1 598058D2
-P 6900 3550
-F 0 "J7" H 6950 3750 50  0000 C CNN
-F 1 "GS3" H 6950 3351 50  0000 C CNN
-F 2 "Connectors:GS3" V 6988 3476 50  0001 C CNN
-F 3 "" H 6900 3550 50  0001 C CNN
-	1    6900 3550
-	0    1    1    0
-$EndComp
-Text Label 7150 1800 2    60   ~ 0
+Text Label 7750 1550 2    60   ~ 0
 D4
 Wire Wire Line
@@
 	3650 2350 3950 2350
 Wire Wire Line
-	3650 1950 3650 2350
+	3650 1900 3650 2350
 Wire Wire Line
 	3650 2150 3400 2150
@@
 Connection ~ 7000 2650
 Wire Wire Line
-	7250 2100 7250 2300
+	7250 1900 7250 2300
 Wire Wire Line
 	7250 2250 6950 2250
@@
 L +3.3V #PWR03
 U 1 1 598062DA
-P 7350 1800
-F 0 "#PWR03" H 7350 1650 50  0001 C CNN
-F 1 "+3.3V" H 7350 1940 50  0000 C CNN
-F 2 "" H 7350 1800 50  0001 C CNN
-F 3 "" H 7350 1800 50  0001 C CNN
-	1    7350 1800
-	1    0    0    -1
-$EndComp
+P 7950 1550
+F 0 "#PWR03" H 7950 1400 50  0001 C CNN
+F 1 "+3.3V" H 7950 1690 50  0000 C CNN
+F 2 "" H 7950 1550 50  0001 C CNN
+F 3 "" H 7950 1550 50  0001 C CNN
+	1    7950 1550
+	1    0    0    -1
+$EndComp
+Wire Wire Line
+	7000 2650 7000 3100
 $Comp
 L +3.3V #PWR04
-U 1 1 5980631F
-P 3750 1650
-F 0 "#PWR04" H 3750 1500 50  0001 C CNN
-F 1 "+3.3V" H 3750 1790 50  0000 C CNN
-F 2 "" H 3750 1650 50  0001 C CNN
-F 3 "" H 3750 1650 50  0001 C CNN
-	1    3750 1650
-	1    0    0    -1
-$EndComp
-$Comp
-L +3.3V #PWR05
-U 1 1 598063DF
-P 7000 3400
-F 0 "#PWR05" H 7000 3250 50  0001 C CNN
-F 1 "+3.3V" H 7000 3540 50  0000 C CNN
-F 2 "" H 7000 3400 50  0001 C CNN
-F 3 "" H 7000 3400 50  0001 C CNN
-	1    7000 3400
-	1    0    0    -1
-$EndComp
-Wire Wire Line
-	7000 2650 7000 3100
-$Comp
-L +3.3V #PWR06
 U 1 1 598068CC
 P 3300 3400
-F 0 "#PWR06" H 3300 3250 50  0001 C CNN
+F 0 "#PWR04" H 3300 3250 50  0001 C CNN
 F 1 "+3.3V" H 3300 3540 50  0000 C CNN
 F 2 "" H 3300 3400 50  0001 C CNN
@@
 $EndComp
 $Comp
-L GND #PWR07
+L GND #PWR05
 U 1 1 59806902
 P 3000 3450
-F 0 "#PWR07" H 3000 3200 50  0001 C CNN
+F 0 "#PWR05" H 3000 3200 50  0001 C CNN
 F 1 "GND" H 3000 3300 50  0000 C CNN
 F 2 "" H 3000 3450 50  0001 C CNN
@@
 $EndComp
 $Comp
-L PWR_FLAG #FLG08
+L PWR_FLAG #FLG06
 U 1 1 59806938
 P 3000 3450
-F 0 "#FLG08" H 3000 3525 50  0001 C CNN
+F 0 "#FLG06" H 3000 3525 50  0001 C CNN
 F 1 "PWR_FLAG" H 3000 3600 50  0000 C CNN
 F 2 "" H 3000 3450 50  0001 C CNN
@@
 $EndComp
 $Comp
-L PWR_FLAG #FLG09
+L PWR_FLAG #FLG07
 U 1 1 598069BA
 P 3300 3400
-F 0 "#FLG09" H 3300 3475 50  0001 C CNN
+F 0 "#FLG07" H 3300 3475 50  0001 C CNN
 F 1 "PWR_FLAG" H 3300 3550 50  0000 C CNN
 F 2 "" H 3300 3400 50  0001 C CNN
@@
 	-1   0    0    1
 $EndComp
-Text Notes 6750 3300 2    60   ~ 0
-D7 as +3.3V
 NoConn ~ 4500 3700
 NoConn ~ 3550 4300
@@
 NoConn ~ 6950 2550
 $Comp
-L GND #PWR010
+L GND #PWR08
 U 1 1 59806FDD
 P 5200 3300
-F 0 "#PWR010" H 5200 3050 50  0001 C CNN
+F 0 "#PWR08" H 5200 3050 50  0001 C CNN
 F 1 "GND" H 5200 3150 50  0000 C CNN
 F 2 "" H 5200 3300 50  0001 C CNN
@@
 Wire Wire Line
 	5400 3300 5400 3400
+$Comp
+L CONN_01X01 J4
+U 1 1 59D60D96
+P 5400 4800
+F 0 "J4" H 5400 4900 50  0000 C CNN
+F 1 "Aloes_Logo" V 5500 4800 50  0000 C CNN
+F 2 "Aloes:Aloes_mini" H 5400 4800 50  0001 C CNN
+F 3 "" H 5400 4800 50  0001 C CNN
+	1    5400 4800
+	1    0    0    -1
+$EndComp
+$Comp
+L CONN_01X01 J6
+U 1 1 59D60EE7
+P 5400 5350
+F 0 "J6" H 5400 5450 50  0000 C CNN
+F 1 "OSHW_Logo" V 5500 5350 50  0000 C CNN
+F 2 "Symbols:OSHW-Logo_5.7x6mm_SilkScreen" H 5400 5350 50  0001 C CNN
+F 3 "" H 5400 5350 50  0001 C CNN
+	1    5400 5350
+	1    0    0    -1
+$EndComp
+Text Label 3550 4400 2    60   ~ 0
+A6
+Text Label 4500 4400 2    60   ~ 0
+A7
+NoConn ~ 4500 4400
+NoConn ~ 3550 4400
+Wire Wire Line
+	7850 1900 7850 1850
+Wire Wire Line
+	3650 1900 7850 1900
+Connection ~ 7250 1900
+Wire Wire Line
+	6900 3700 7550 3700
+Wire Wire Line
+	7550 3700 7550 1900
+Connection ~ 7550 1900
+NoConn ~ 3550 3900
+NoConn ~ 3550 4100
+NoConn ~ 5200 4800
+NoConn ~ 5200 5350
 $EndSCHEMATC
