File: Cosmonode_ext04/Cosmonode_ext_04.sch (KiCad schematic (older format))
At the start: 24 parts, among them J1 PT100, J2 CONN_01X07, J3 CONN_01X07, J4 GS3, J5 GS3, U1 TL431ACDBZR, U2 LMV321, U3 RT9193-30PB

Commit message: fully update to v0.3
Parts:
- added J6: Aloes_Logo, Aloes:Aloes_mini, symbol CONN_01X01
- added J7: OSHW_Logo, Symbols:OSHW-Logo_5.7x6mm_SilkScreen, symbol CONN_01X01
- J1: footprint Connectors_JST:JST_PH_B3B-PH-K_03x2.00mm_Straight -> Connectors_JST:JST_XH_B03B-XH-A_03x2.50mm_Straight
- J2, J3: value CONN_01X07 -> CONN_01X08; footprint Pin_Headers:Pin_Header_Straight_1x07_Pitch2.54mm -> Socket_Strips:Socket_Strip_Straight_1x08_Pitch2.54mm; symbol CONN_01X07 -> CONN_01X08
Connections:
- new net A6: J2.8 (P8)
- new net A7: J3.8 (P8)
- no-connect marks 7 -> 11
Changed lines of the file:
@@
 LIBS:RT9193-30PB
 LIBS:TL431ACDBZR
+LIBS:Cosmonode_ext_04-cache
 EELAYER 25 0
 EELAYER END
@@
 F 0 "J1" H 3650 5300 50  0000 C CNN
 F 1 "PT100" V 3750 5100 50  0000 C CNN
-F 2 "Connectors_JST:JST_PH_B3B-PH-K_03x2.00mm_Straight" H 3650 5100 50  0001 C CNN
+F 2 "Connectors_JST:JST_XH_B03B-XH-A_03x2.50mm_Straight" H 3650 5100 50  0001 C CNN
 F 3 "" H 3650 5100 50  0001 C CNN
 	1    3650 5100
@@
 +3.0V
 $Comp
-L CONN_01X07 J3
+L CONN_01X08 J3
 U 1 1 59825EDD
-P 8450 4550
-F 0 "J3" H 8450 4950 50  0000 C CNN
-F 1 "CONN_01X07" V 8550 4550 50  0000 C CNN
-F 2 "Pin_Headers:Pin_Header_Straight_1x07_Pitch2.54mm" H 8450 4550 50  0001 C CNN
-F 3 "" H 8450 4550 50  0001 C CNN
-	1    8450 4550
-	1    0    0    -1
-$EndComp
-$Comp
-L CONN_01X07 J2
+P 8450 4600
+F 0 "J3" H 8450 5000 50  0000 C CNN
+F 1 "CONN_01X08" V 8550 4600 50  0000 C CNN
+F 2 "Socket_Strips:Socket_Strip_Straight_1x08_Pitch2.54mm" H 8450 4600 50  0001 C CNN
+F 3 "" H 8450 4600 50  0001 C CNN
+	1    8450 4600
+	1    0    0    -1
+$EndComp
+$Comp
+L CONN_01X08 J2
 U 1 1 59825F9E
-P 7550 4550
-F 0 "J2" H 7550 4950 50  0000 C CNN
-F 1 "CONN_01X07" V 7650 4550 50  0000 C CNN
-F 2 "Pin_Headers:Pin_Header_Straight_1x07_Pitch2.54mm" H 7550 4550 50  0001 C CNN
-F 3 "" H 7550 4550 50  0001 C CNN
-	1    7550 4550
+P 7550 4600
+F 0 "J2" H 7550 5000 50  0000 C CNN
+F 1 "CONN_01X08" V 7650 4600 50  0000 C CNN
+F 2 "Socket_Strips:Socket_Strip_Straight_1x08_Pitch2.54mm" H 7550 4600 50  0001 C CNN
+F 3 "" H 7550 4600 50  0001 C CNN
+	1    7550 4600
 	1    0    0    -1
 $EndComp
@@
 	5850 4200 5850 4150
 Connection ~ 5850 4150
+$Comp
+L CONN_01X01 J6
+U 1 1 59D4B1E8
+P 7350 5550
+F 0 "J6" H 7350 5650 50  0000 C CNN
+F 1 "Aloes_Logo" V 7450 5550 50  0000 C CNN
+F 2 "Aloes:Aloes_mini" H 7350 5550 50  0001 C CNN
+F 3 "" H 7350 5550 50  0001 C CNN
+	1    7350 5550
+	1    0    0    -1
+$EndComp
+$Comp
+L CONN_01X01 J7
+U 1 1 59D4B315
+P 7350 6000
+F 0 "J7" H 7350 6100 50  0000 C CNN
+F 1 "OSHW_Logo" V 7450 6000 50  0000 C CNN
+F 2 "Symbols:OSHW-Logo_5.7x6mm_SilkScreen" H 7350 6000 50  0001 C CNN
+F 3 "" H 7350 6000 50  0001 C CNN
+	1    7350 6000
+	1    0    0    -1
+$EndComp
+NoConn ~ 7150 5550
+NoConn ~ 7150 6000
+Text Label 7350 4950 2    60   ~ 0
+A6
+Text Label 8250 4950 2    60   ~ 0
+A7
+NoConn ~ 8250 4950
+NoConn ~ 7350 4950
 $EndSCHEMATC
