File: Cosmonode_ext05/Cosmonode_ext05.sch (KiCad schematic (older format))
At the start: 16 parts, among them J1 CH340G, J2 GS2, J3 USB_OTG, J4 CONN_01X08, J5 CONN_01X08, J6 CONN_02X05, J7 CONN_01X09, Y1 Crystal_GND2

Commit message: big push!
Parts:
- removed J2: GS2, Connectors:GS2, symbol GS2
- added J2: OSWH_Logo, Symbols:OSHW-Logo_5.7x6mm_SilkScreen, symbol CONN_01X01
- added J8: Aloes_Logo, Aloes:Aloes_mini, symbol CONN_01X01
- C1, C2: footprint Capacitors_SMD:C_0402_NoSilk -> Capacitors_SMD:C_0603_HandSoldering
- R1, R2, R3, R4: footprint Resistors_SMD:R_0402_NoSilk -> Resistors_SMD:R_0603_HandSoldering
Connections:
- net DTR_1 renamed AREF
- net DTR_2: no longer names the net of J1.13 (DTR)
- no-connect marks 21 -> 25
Changed lines of the file:
@@
 LIBS:RT9193-30PB
 LIBS:SI7020-A20-YM0R
-LIBS:SMD-RESONATOR-8MHZ-33PF-0.1__3P-3.2X1.3MM_
 LIBS:TL431ACDBZR
-LIBS:TSL2561T_6P-3.8X2.6MM_
 LIBS:wemos_mini
-LIBS:XC6206P302MR_SOT23_
-LIBS:Cosmonode_ext05_v03-cache
+LIBS:Cosmonode_ext05-cache
 EELAYER 25 0
 EELAYER END
@@
 Rev ""
 Comp ""
-Comment1 ""
+Comment1 "Extension #5 ISP header - USB to TTL"
 Comment2 ""
 Comment3 ""
@@
 F 0 "C1" H 2460 2820 50  0000 L CNN
 F 1 "100nF" H 2460 2670 50  0000 L CNN
-F 2 "Capacitors_SMD:C_0402_NoSilk" H 2450 2750 50  0001 C CNN
+F 2 "Capacitors_SMD:C_0603_HandSoldering" H 2450 2750 50  0001 C CNN
 F 3 "" H 2450 2750 50  0001 C CNN
 	1    2450 2750
@@
 F 0 "C2" H 5010 2020 50  0000 L CNN
 F 1 "100nF" H 5010 1870 50  0000 L CNN
-F 2 "Capacitors_SMD:C_0402_NoSilk" H 5000 1950 50  0001 C CNN
+F 2 "Capacitors_SMD:C_0603_HandSoldering" H 5000 1950 50  0001 C CNN
 F 3 "" H 5000 1950 50  0001 C CNN
 	1    5000 1950
@@
 F 0 "R2" V 5780 1200 50  0000 C CNN
 F 1 "1K" V 5700 1200 50  0000 C CNN
-F 2 "Resistors_SMD:R_0402_NoSilk" V 5630 1200 50  0001 C CNN
+F 2 "Resistors_SMD:R_0603_HandSoldering" V 5630 1200 50  0001 C CNN
 F 3 "" H 5700 1200 50  0001 C CNN
 	1    5700 1200
@@
 F 0 "R3" V 6480 1200 50  0000 C CNN
 F 1 "5k" V 6400 1200 50  0000 C CNN
-F 2 "Resistors_SMD:R_0402_NoSilk" V 6330 1200 50  0001 C CNN
+F 2 "Resistors_SMD:R_0603_HandSoldering" V 6330 1200 50  0001 C CNN
 F 3 "" H 6400 1200 50  0001 C CNN
 	1    6400 1200
@@
 F 0 "R4" V 6480 1400 50  0000 C CNN
 F 1 "5k" V 6400 1400 50  0000 C CNN
-F 2 "Resistors_SMD:R_0402_NoSilk" V 6330 1400 50  0001 C CNN
+F 2 "Resistors_SMD:R_0603_HandSoldering" V 6330 1400 50  0001 C CNN
 F 3 "" H 6400 1400 50  0001 C CNN
 	1    6400 1400
@@
 F 0 "R1" V 5730 1400 50  0000 C CNN
 F 1 "1k" V 5650 1400 50  0000 C CNN
-F 2 "Resistors_SMD:R_0402_NoSilk" V 5580 1400 50  0001 C CNN
+F 2 "Resistors_SMD:R_0603_HandSoldering" V 5580 1400 50  0001 C CNN
 F 3 "" H 5650 1400 50  0001 C CNN
 	1    5650 1400
@@
 Text Label 6100 1900 0    60   ~ 0
 TX
-Text Label 4350 2050 0    60   ~ 0
-DTR_2
 Text Label 2000 2150 0    60   ~ 0
 USB_P
@@
 SCK
 Text Label 7450 4100 2    60   ~ 0
-DTR_1
+AREF
 $Comp
 L VCC #PWR015
@@
 	1    0    0    -1
 $EndComp
-Text Label 5800 2500 2    60   ~ 0
-DTR_2
-Text Label 6200 2500 0    60   ~ 0
-DTR_1
-$Comp
-L GS2 J2
-U 1 1 59CD95B9
-P 6000 2500
-F 0 "J2" H 6100 2650 50  0000 C CNN
-F 1 "GS2" H 6100 2351 50  0000 C CNN
-F 2 "Connectors:GS2" V 6074 2500 50  0001 C CNN
-F 3 "" H 6000 2500 50  0001 C CNN
-	1    6000 2500
-	0    1    1    0
-$EndComp
+NoConn ~ 7450 4100
+NoConn ~ 4350 2050
+$Comp
+L Logo_Open_Hardware_Small #LOGO1
+U 1 1 59D12DEC
+P 10800 6850
+F 0 "#LOGO1" H 10800 7125 50  0001 C CNN
+F 1 "Logo_Open_Hardware_Small" H 10800 6625 50  0001 C CNN
+F 2 "" H 10800 6850 50  0001 C CNN
+F 3 "" H 10800 6850 50  0001 C CNN
+	1    10800 6850
+	1    0    0    -1
+$EndComp
+$Comp
+L CONN_01X01 J2
+U 1 1 59D12ED6
+P 4150 4900
+F 0 "J2" H 4150 5000 50  0000 C CNN
+F 1 "OSWH_Logo" V 4250 4900 50  0000 C CNN
+F 2 "Symbols:OSHW-Logo_5.7x6mm_SilkScreen" H 4150 4900 50  0001 C CNN
+F 3 "" H 4150 4900 50  0001 C CNN
+	1    4150 4900
+	1    0    0    -1
+$EndComp
+$Comp
+L CONN_01X01 J8
+U 1 1 59D15050
+P 4150 4400
+F 0 "J8" H 4150 4500 50  0000 C CNN
+F 1 "Aloes_Logo" V 4250 4400 50  0000 C CNN
+F 2 "Aloes:Aloes_mini" H 4150 4400 50  0001 C CNN
+F 3 "" H 4150 4400 50  0001 C CNN
+	1    4150 4400
+	1    0    0    -1
+$EndComp
+NoConn ~ 3950 4400
+NoConn ~ 3950 4900
 $EndSCHEMATC

Commit message: big push2
Parts:
- Y1: footprint SMD-RESONATOR-8MHZ-33PF-0.1__3P-3.2X1.3MM_:X3-SMD-3.6X1.3X0.8MM -> SMD-RESONATOR-8MHZ-33PF:X3-SMD-3.6X1.3X0.8MM
Changed lines of the file:
@@
 F 0 "Y1" H 3450 3275 50  0000 C CNN
 F 1 "Crystal_GND2" H 3450 3200 50  0000 C CNN
-F 2 "SMD-RESONATOR-8MHZ-33PF-0.1__3P-3.2X1.3MM_:X3-SMD-3.6X1.3X0.8MM" H 3450 3050 50  0001 C CNN
+F 2 "SMD-RESONATOR-8MHZ-33PF:X3-SMD-3.6X1.3X0.8MM" H 3450 3050 50  0001 C CNN
 F 3 "" H 3450 3050 50  0001 C CNN
 	1    3450 3050

Commit message: update to v0.5 ( base, ext05, ext07, ext08 )
Parts:
- added C3, C4: 100nF, Capacitors_SMD:C_0603_HandSoldering, symbol C_Small
- added D3: 0603, LEDs:LED_0603, symbol LED
- added D4, D5: MBR0520, Diodes_SMD:D_SOD-123, symbol MBR0520
- added JP1: Jumper_NC_Dual, Pin_Headers:Pin_Header_Straight_1x03_Pitch2.54mm, symbol Jumper_NC_Dual
- C1: value 100nF -> 10uF
- J4: value CONN_01X08 -> CONN_01X12; footprint Socket_Strips:Socket_Strip_Straight_1x08_Pitch2.54mm -> Socket_Strips:Socket_Strip_Straight_1x12_Pitch2.54mm; symbol CONN_01X08 -> CONN_01X12
- J5: value CONN_01X08 -> CONN_01X05; footprint Socket_Strips:Socket_Strip_Straight_1x08_Pitch2.54mm -> Socket_Strips:Socket_Strip_Straight_1x05_Pitch2.54mm; symbol CONN_01X08 -> CONN_01X05
- J7: value CONN_01X09 -> CONN_01X12; footprint Socket_Strips:Socket_Strip_Straight_1x09_Pitch2.54mm -> Socket_Strips:Socket_Strip_Straight_1x12_Pitch2.54mm; symbol CONN_01X09 -> CONN_01X12
- R1: value 1k -> 1k5
- R2: value 1K -> 1k5
- R3, R4: value 5k -> 1k5
- Y1: value Crystal_GND2 -> CSTCE12M0V53-R0
Connections:
- net AREF is gone; now on net RX: J7.9 (P9)
- net A0: now also J7.1 (P1); no longer J5.6 (P6)
- net A1: now also J7.2 (P2); no longer J5.7 (P7)
- net A4: now also J7.4 (P4); no longer J4.6 (P6)
- net A5: now also J7.5 (P5); no longer J4.7 (P7)
- net A6: now also J7.6 (P6); no longer J5.8 (P8)
- net A7: now also J7.7 (P7); no longer J4.8 (P8)
- net D3: now also J7.11 (P11); no longer J5.1 (P1)
- net D4: now also J7.12 (P12); no longer J5.2 (P2)
- net D5: now also J4.4 (P4); no longer J5.3 (P3)
- net D6: now also J4.5 (P5); no longer J5.4 (P4)
- net D7: now also J4.6 (P6); no longer J5.5 (P5)
- net GND: now also J4.3 (P3), J5.2 (P2), R1.1, C3.2, C4.2; no longer J4.4 (P4), J4.5 (P5), J7.8 (P8)
- net MISO: now also J4.11 (P11); no longer J7.5 (P5)
- net MOSI: now also J4.10 (P10); no longer J7.4 (P4)
- net RST: now also J4.9 (P9); no longer J7.1 (P1)
- net RX: now also D1.1 (K), J1.3 (RxD), J5.3 (P3); no longer J7.2 (P2), R2.1, R3.2
- net SCK: now also J4.12 (P12); no longer J7.6 (P6)
- net TX: now also D2.1 (K), J1.2 (TxD), J7.8 (P8), R2.1; no longer J7.3 (P3), R1.1, R4.2
- net DTR: now reaches J1.13 (DTR)
- net DTR: now also J5.5 (P5)
- net at R1.2: now also D3.1 (K); no longer J1.2 (TxD)
- net at R2.2: now also J5.4 (P4); no longer J1.3 (RxD)
- net +3V3: now reaches J1.4 (3V)
- net +3V3: now also J4.2 (P2), J5.1 (P1), J6.2 (P2), C3.1, JP1.1; no longer C1.1
- net at R3.1: now also D1.2 (A); no longer D1.1 (K)
- net at R4.1: now also D2.2 (A); no longer D2.1 (K)
- net BAT+ renamed +BATT
- removed net VCC: C2.1, D1.2 (A), D2.2 (A), J1.16 (VCC), J3.1 (VBUS), J4.2 (P2), J4.3 (P3), J6.2 (P2), J7.7 (P7)
- new net: C4.1, D3.2 (A), D5.1 (K), J1.16 (VCC), JP1.2, R3.2, R4.2
- new net: D4.1 (K), D5.2 (A)
- new net +5V: C1.1, C2.1, D4.2 (A), J3.1 (VBUS), JP1.3
- new net A3: J7.3 (P3)
- new net D2: J7.10 (P10)
- new net D8: J4.7 (P7)
- new net D9: J4.8 (P8)
- no-connect marks 25 -> 27
Other:
- moved on the sheet: D1, D2, J1, J2, J3, J6, J8, R3, R4, Y1
