File: Cosmonode_ext07/Cosmonode_ext07.sch (KiCad schematic (older format))
At the start: 9 parts, among them J1 OSHW_Logo, J2 MH-Z19, J3 CONN_01X08, J4 CONN_01X08, J5 GS3, J6 GS3, J7 Aloes_Logo, J8 CONN_01X09, U1 XC6206P502MR

Commit message: update to v0.5 ( base, ext05, ext07, ext08 )
Parts:
- removed J8: CONN_01X09, Pin_Headers:Pin_Header_Straight_1x09_Pitch2.54mm, symbol CONN_01X09
- added J8: CONN_01X04, symbol CONN_01X04
- added J9: CONN_01X05, symbol CONN_01X05
- J3, J4: value CONN_01X08 -> CONN_01X12; footprint Pin_Headers:Pin_Header_Straight_1x08_Pitch2.54mm -> Pin_Headers:Pin_Header_Straight_1x12_Pitch2.54mm; symbol CONN_01X08 -> CONN_01X12
Connections:
- net +3V3: no longer J4.3 (P3)
- net +5V: now also J8.4 (P4)
- net A0: now also J2.3 (TX), J3.1 (P1), J9.3 (P3); no longer J3.6 (P6)
- net A1: now also J2.2 (RX), J3.2 (P2), J9.2 (P2); no longer J3.7 (P7)
- net A4: now also J3.4 (P4); no longer J4.6 (P6)
- net A5: now also J3.5 (P5); no longer J4.7 (P7)
- net A6: now also J3.6 (P6); no longer J3.8 (P8)
- net D3: now also J3.11 (P11); no longer J3.1 (P1)
- net D4: now also J3.12 (P12); no longer J3.2 (P2)
- net D5: now also J4.4 (P4); no longer J3.3 (P3)
- net D6: now also J4.5 (P5); no longer J3.4 (P4)
- net D7: now also J4.6 (P6); no longer J3.5 (P5)
- net GND: now also J2.7 (GND), J4.3 (P3); no longer J4.4 (P4), J4.5 (P5)
- net MISO: now also J4.11 (P11)
- net MOSI: now also J4.10 (P10)
- net RST: now also J4.9 (P9)
- net RX: now also J3.8 (P8); no longer J2.2 (RX)
- net SCK: now also J4.12 (P12)
- net TX: now also J3.9 (P9); no longer J2.3 (TX)
- net at J6.2 (G2): now also J8.3 (P3); no longer J2.7 (GND)
- net AREF renamed D9
- net BAT+ renamed +BATT
- new net A3: J3.3 (P3)
- new net A7: J3.7 (P7)
- new net D2: J3.10 (P10)
- new net D8: J4.7 (P7)
- no-connect marks 13 -> 27
Other:
- moved on the sheet: J2
