File: Cosmonode_ext03/Cosmonode_ext03.sch (KiCad schematic (older format))
At the start: 6 parts, among them J1 CONN_01X04, J2 GS3, J3 GS3, J4 CONN_01X04, J5 CONN_01X08, J6 CONN_01X08

Commit message: big push2
Parts:
- added J7: Aloes_Logo, Aloes:Aloes_mini, symbol CONN_01X01
- added J8: OSHW_Logo, Symbols:OSHW-Logo_5.7x6mm_SilkScreen, symbol CONN_01X01
Changed lines of the file:
@@
 LIBS:valves
 LIBS:BSS138
-LIBS:XC6206P302MR_SOT23_
 LIBS:Cosmonode_ext03-cache
 EELAYER 25 0
@@
 NoConn ~ 6100 2700
 NoConn ~ 6100 2800
+$Comp
+L CONN_01X01 J7
+U 1 1 59D34FA9
+P 4450 4750
+F 0 "J7" H 4450 4850 50  0000 C CNN
+F 1 "Aloes_Logo" V 4550 4750 50  0000 C CNN
+F 2 "Aloes:Aloes_mini" H 4450 4750 50  0001 C CNN
+F 3 "" H 4450 4750 50  0001 C CNN
+	1    4450 4750
+	1    0    0    -1
+$EndComp
+$Comp
+L CONN_01X01 J8
+U 1 1 59D42085
+P 5050 4750
+F 0 "J8" H 5050 4850 50  0000 C CNN
+F 1 "OSHW_Logo" V 5150 4750 50  0000 C CNN
+F 2 "Symbols:OSHW-Logo_5.7x6mm_SilkScreen" H 5050 4750 50  0001 C CNN
+F 3 "" H 5050 4750 50  0001 C CNN
+	1    5050 4750
+	1    0    0    -1
+$EndComp
 $EndSCHEMATC

Commit message: update to V0.7 (WIP)
Parts:
- removed J1, J4: CONN_01X04, Connectors_JST:JST_XH_B04B-XH-A_04x2.50mm_Straight, symbol CONN_01X04
- removed J2, J3: GS3, Connectors:GS3, symbol GS3
- removed J8: OSHW_Logo, Symbols:OSHW-Logo_5.7x6mm_SilkScreen, symbol CONN_01X01
- added J1: OSHW_Logo, Symbols:OSHW-Logo_5.7x6mm_SilkScreen, symbol CONN_01X01
- added J10, J11, J5, J6: CONN_01X03, Pin_Headers:Pin_Header_Straight_1x03_Pitch2.54mm, symbol CONN_01X03
- added J12: CONN_02X03, Pin_Headers:Pin_Header_Straight_2x03_Pitch2.54mm, symbol CONN_02X03
- added J13: CONN_02X09, Pin_Headers:Pin_Header_Straight_2x09_Pitch2.54mm, symbol CONN_02X09
- added J2, J8, J9: CONN_01X04, Pin_Headers:Pin_Header_Straight_1x04_Pitch2.54mm, symbol CONN_01X04
- J3: renamed from J5; value CONN_01X08 -> CONN_01X12; footprint Socket_Strips:Socket_Strip_Straight_1x08_Pitch2.54mm -> Socket_Strips:Socket_Strip_Straight_1x12_Pitch2.54mm; symbol CONN_01X08 -> CONN_01X12
- J4: renamed from J6; value CONN_01X08 -> CONN_01X12; footprint Socket_Strips:Socket_Strip_Straight_1x08_Pitch2.54mm -> Socket_Strips:Socket_Strip_Straight_1x12_Pitch2.54mm; symbol CONN_01X08 -> CONN_01X12
Connections:
- net +3V3: now also J10.1 (P1), J11.1 (P1), J12.1 (P1), J12.3 (P3), J12.5 (P5), J2.1 (P1), J5.1 (P1), J6.1 (P1), J8.1 (P1), J9.1 (P1); no longer J4.3 (P3)
- net A0: now also J3.1 (P1), J10.2 (P2); no longer J3.6 (P6)
- net A1: now also J3.2 (P2), J11.2 (P2); no longer J3.7 (P7)
- net A4: now also J3.4 (P4), J2.2 (P2), J8.2 (P2); no longer J4.6 (P6)
- net A5: now also J3.5 (P5), J2.3 (P3), J8.3 (P3); no longer J4.7 (P7)
- net A6: now also J3.6 (P6); no longer J3.8 (P8)
- net A7: now also J3.7 (P7); no longer J4.8 (P8)
- net D3: now also J3.11 (P11), J6.2 (P2); no longer J3.1 (P1)
- net D4: now also J3.12 (P12), J5.2 (P2); no longer J3.2 (P2)
- net D5: now also J4.4 (P4); no longer J3.3 (P3)
- net D6: now also J4.5 (P5), J9.2 (P2); no longer J3.4 (P4)
- net D7: now also J4.6 (P6), J9.3 (P3); no longer J3.5 (P5)
- net GND: now also J4.3 (P3), J10.3 (P3), J11.3 (P3), J12.2 (P2), J12.4 (P4), J12.6 (P6), J2.4 (P4), J5.3 (P3), J6.3 (P3), J8.4 (P4), J9.4 (P4); no longer J4.4 (P4), J4.5 (P5)
- net BAT+ renamed +BATT
- new net A3: J3.3 (P3)
- new net D2: J3.10 (P10)
- new net D8: J4.7 (P7)
- new net D9: J4.8 (P8)
- new net MISO: J4.11 (P11)
- new net MOSI: J4.10 (P10)
- new net RST: J4.9 (P9)
- new net RX: J3.8 (P8)
- new net SCK: J4.12 (P12)
- new net TX: J3.9 (P9)
- no-connect marks 8 -> 33
Other:
- note added: "Shield for cosmonode\nProtoboard"
- note removed: "Shield for cosmonode\nConnection to 5V XKC YV sensor"
