File: Cosmonode/Cosmonode.sch (KiCad schematic (older format))
At the start: 30 parts, among them J1 CONN_01X07, J2 CONN_01X07, J3 CONN_01X02, J4 CONN_01X01, J5 CONN_01X06, SW1 SW_DIP_x01, U1 ATMEGA328P-AU, U2 RFM69CW, U3 M25P40, U4 XC6206P332MR, U6 ATSHA204, Y2 Crystal_GND2

Commit message: micro update
Other:
- note added: "Does not work, to update!"
- note removed: "Really useful ?"
Changed lines of the file:
@@
 	4050 4450 3950 4450
 Text Notes 4750 2800 2    60   ~ 0
-Really useful ?
+Does not work, to update!
 Text Label 10450 900  2    60   ~ 0
 BAT+

Commit message: new version 0.3
Parts:
- added U5: NRF24L01_Breakout, mysensors_radios:NRF24L01-SMD, symbol NRF24L01_Breakout
- J1, J2: value CONN_01X07 -> CONN_01X08; footprint Socket_Strips:Socket_Strip_Straight_1x07_Pitch2.54mm -> Pin_Headers:Pin_Header_Straight_1x08_Pitch2.54mm; symbol CONN_01X07 -> CONN_01X08
- J5: value CONN_01X06 -> CONN_01X09; footprint Pin_Headers:Pin_Header_Straight_1x06_Pitch2.54mm -> Pin_Headers:Pin_Header_Straight_1x09_Pitch2.54mm; symbol CONN_01X06 -> CONN_01X09
Connections:
- wire segments 78 -> 81
- no-connect marks 8 -> 7
Other:
- note removed: "Does not work, to update!"
- moved on the sheet: SW1

Commit message: big push!
Parts:
- added J10: WEEE_Logo, Symbols:WEEE-Logo_4.2x6mm_SilkScreen, symbol CONN_01X01
- added J11: Aloes_Logo, Aloes:Aloes, symbol CONN_01X01
- added J12: Aloes_mini_Logo, Aloes:Aloes_mini, symbol CONN_01X01
- added J6: GS3, Connectors:GS3, symbol GS3
- J4: value CONN_01X01 -> OSHW; footprint Symbols:OSHW-Logo2_7.3x6mm_SilkScreen -> Symbols:OSHW-Logo_7.5x8mm_Copper
- Y1: renamed from Y2; footprint SMD-RESONATOR-8MHZ-33PF-0.1__3P-3.2X1.3MM_:X3-SMD-3.6X1.3X0.8MM -> SMD-RESONATOR-8MHZ-33PF:X3-SMD-3.6X1.3X0.8MM
- renumbered C2 to C1, C4 to C2, C6 to C3, C7 to C4, C9 to C5, C10 to C6, C1 to C7, C12 to C8, J5 to J3, J3 to J5, R3 to R1, R4 to R2, R5 to R3, R10 to R4, R11 to R5, R13 to R6, R14 to R7, R1 to R8, R2 to R9, U5 to U3, U3 to U4, U4 to U5
Connections:
- net DTR is gone; now on net GND: C3.2, J3.9 (P9)
- net +3V3: now also J6.2 (G2); no longer U2.9 (3.3V), U3.2 (VCC)
- new net VCC_NRF24: J6.1 (G1), U3.2 (VCC)
- new net VCC_RFM69: J6.3 (G3), U2.9 (3.3V)
Other:
- moved on the sheet: C1, C2, C3, J4, R1, R2, R3, SW1, U1, Y1

Commit message: big push2
Connections:
- net GND: no longer J3.9 (P9)
- net AREF: now reaches C2.2, U1.20 (AREF)
- net AREF: now also J3.9 (P9)
Changed lines of the file:
@@
 P 1350 1750
 F 0 "C2" H 1360 1820 50  0000 L CNN
-F 1 "100nF" H 1360 1670 50  0000 L CNN
+F 1 "100nF" V 1250 1650 50  0000 L CNN
 F 2 "Capacitors_SMD:C_0603_HandSoldering" H 1350 1750 50  0001 C CNN
 F 3 "" H 1350 1750 50  0001 C CNN
@@
 	4450 2600 4450 2700
 Connection ~ 4450 2600
-Text Label 1050 1750 2    60   ~ 0
-AREF
 Connection ~ 1150 1750
 $Comp
@@
 Wire Wire Line
 	6100 2350 6100 2300
+Text Label 1550 1650 2    60   ~ 0
+AREF
+Wire Wire Line
+	1550 1750 1550 1650
+Connection ~ 1550 1750
 $EndSCHEMATC

Commit message: fix before test
Parts:
- added J7: Kicad_Logo, Symbols:KiCad-Logo2_6mm_SilkScreen, symbol CONN_01X01
Changed lines of the file:
@@
 	1550 1750 1550 1650
 Connection ~ 1550 1750
+$Comp
+L CONN_01X01 J7
+U 1 1 59D61A7D
+P 2050 6950
+F 0 "J7" H 2050 7050 50  0000 C CNN
+F 1 "Kicad_Logo" V 2150 6950 50  0000 C CNN
+F 2 "Symbols:KiCad-Logo2_6mm_SilkScreen" H 2050 6950 50  0001 C CNN
+F 3 "" H 2050 6950 50  0001 C CNN
+	1    2050 6950
+	1    0    0    -1
+$EndComp
 $EndSCHEMATC

Commit message: update to v0.5 ( base, ext05, ext07, ext08 )
Parts:
- removed J3: CONN_01X09, Pin_Headers:Pin_Header_Straight_1x09_Pitch2.54mm, symbol CONN_01X09
- removed J6: GS3, Connectors:GS3, symbol GS3
- removed J7: Kicad_Logo, Symbols:KiCad-Logo2_6mm_SilkScreen, symbol CONN_01X01
- removed U3: NRF24L01_Breakout, mysensors_radios:NRF24L01-SMD, symbol NRF24L01_Breakout
- added C9: 100nF, Capacitors_SMD:C_0603_HandSoldering, symbol C_Small
- added D1, D2: MBR0520, Diodes_SMD:D_SOD-123, symbol LL4148
- added D3, D4, D5: LED, LEDs:LED_0603_HandSoldering, symbol LED
- added J13: CONN_01X05, Pin_Headers:Pin_Header_Straight_1x05_Pitch2.54mm, symbol CONN_01X05
- added J14, J3, J9: GS2, Connectors:GS2, symbol GS2
- added J8: USB_OTG, Connectors_USB:USB_Micro-B_Molex-105017-0001, symbol USB_OTG
- added P1: COAX, sma:EDGE_SMA_5, symbol COAX
- added Q1: BSS123, TO_SOT_Packages_SMD:TSOT-23, symbol BSS123
- added R10: 10k, Resistors_SMD:R_0603_HandSoldering, symbol R
- added R11: R, Resistors_SMD:R_0603_HandSoldering, symbol R
- added R12, R13, R14: 1k, Resistors_SMD:R_0603_HandSoldering, symbol R
- added U3: RN2483, RN2483:RN2483, symbol RN2483
- added U7: MCP73811T-420I/OT, TO_SOT_Packages_SMD:SOT-23-5_HandSoldering, symbol MCP73811T-420I/OT
- C4, C5: footprint Capacitors_Tantalum_SMD:CP_Tantalum_Case-A_EIA-3216-18_Hand -> Capacitors_Tantalum_SMD:CP_Tantalum_Case-A_EIA-3216-18_Reflow
- J1, J2: value CONN_01X08 -> CONN_01X12; footprint Pin_Headers:Pin_Header_Straight_1x08_Pitch2.54mm -> Pin_Headers:Pin_Header_Straight_1x12_Pitch2.54mm; symbol CONN_01X08 -> CONN_01X12
Connections:
- net VCC_RFM69 is gone; now on net +3V3: U2.9 (3.3V)
- net +3V3: now also C9.1, J13.1 (P1), U3.12 (VDD), U3.34 (VDD); no longer J2.3 (P3)
- net A0: now also J1.1 (P1); no longer J1.6 (P6)
- net A1: now also J1.2 (P2); no longer J1.7 (P7)
- net A3: now also J1.3 (P3)
- net A4: now also J1.4 (P4); no longer J2.6 (P6)
- net A5: now also J1.5 (P5); no longer J2.7 (P7)
- net A6: now also J1.6 (P6); no longer J1.8 (P8)
- net A7: now also J1.7 (P7); no longer J2.8 (P8)
- net D10: now also J9.2 (G2)
- net D2: now also J1.10 (P10)
- net D3: now also J1.11 (P11), U3.6 (UART_TX); no longer J1.1 (P1)
- net D4: now also J1.12 (P12), U3.7 (UART_RX); no longer J1.2 (P2)
- net D5: now also J2.4 (P4), J3.2 (G2); no longer J1.3 (P3)
- net D6: now also J2.5 (P5); no longer J1.4 (P4)
- net D7: now also J2.6 (P6); no longer J1.5 (P5)
- net D8: now also J2.7 (P7), J14.2 (G2)
- net D9: now also J2.8 (P8)
- net GND: now also J2.3 (P3), C9.2, D4.1 (K), D5.1 (K), J13.2 (P2), J8.5 (GND), J8.6 (Shield), P1.2 (GND), Q1.2 (S), R10.2, R11.1, U3.1 (GND), U3.11 (GND), U3.20 (GND), U3.21 (GND), U3.22 (GND), U3.24 (GND), U3.26 (GND), U3.27 (GND), U3.28 (GND), U3.33 (GND), U3.41 (GND), U3.47 (GND), U3.8 (GND), U7.2 (VSS); no longer C3.2, J2.4 (P4), J2.5 (P5)
- net MISO: now also J2.11 (P11)
- net MOSI: now also J2.10 (P10)
- net RST: now also J2.9 (P9)
- net RX: now also J1.8 (P8), J13.3 (P3)
- net SCK: now also J2.12 (P12)
- net TX: now also J1.9 (P9), J13.4 (P4)
- net BAT+ renamed +BATT
- net +BATT: now also D2.2 (A), U7.3 (VBAT); no longer C4.1, C5.1, U5.3 (VIN)
- new net: C4.1, C5.1, D1.1 (K), D2.1 (K), R12.2, U5.3 (VIN), U7.4 (VDD)
- new net: P1.1 (RF), U3.23 (RFH)
- new net: D3.1 (K), U7.1 (CEN)
- new net: R11.2, U7.5 (PROG)
- new net: J3.1 (G1), Q1.1 (G), R10.1
- new net: D3.2 (A), R12.1
- new net: D5.2 (A), R14.1
- new net: J14.1 (G1), R14.2
- new net: D4.2 (A), R13.1
- new net: J9.1 (G1), R13.2
- new net DTR: C3.2, J13.5 (P5)
- new net RADIO_RESET: Q1.3 (D), U3.32 (/RESET)
- new net VDD: D1.2 (A), J8.1 (VBUS)
- no-connect marks 7 -> 40
Other:
- note added: "CPU"
- note added: "Charger Regulation - R11\n10K = 100mA\n5K = 200mA\n2K = 500mA\n1K = 1000mA"
- note added: "Cosmonode v0.5\nATmega328p\nRFM69 or RN 2483 ( both 868Mhz Radio )"
- note added: "RADIO"
- note added: "User LED RX ( red )"
- note added: "User LED TX ( blue )"
- note removed: "CPU & RADIO"
- moved on the sheet: C4, C5, C6, C7, J10, J11, J12, J4, J5, MK1, R4, R5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

Commit message: update to V0.7 (WIP)
Parts:
- removed Q1: BSS123, TO_SOT_Packages_SMD:TSOT-23, symbol BSS123
- removed R10, R2: 10k, Resistors_SMD:R_0603_HandSoldering, symbol R
- removed U4: M25P40, Housings_SOIC:SOIC-8_3.9x4.9mm_Pitch1.27mm, symbol M25P40
- added J6: GS2, Connectors:GS2, symbol GS2
- added JP1: Jumper_NO_Small, Pin_Headers:Pin_Header_Straight_1x02_Pitch2.54mm, symbol Jumper_NO_Small
Connections:
- net A6: now also J9.2 (G2)
- net A7: now also J14.2 (G2)
- net ANT: now also P1.1 (RF), U3.23 (RFH)
- net D10: now also U3.7 (UART_RX); no longer J9.2 (G2)
- net D3: now also J6.1 (G1); no longer U3.6 (UART_TX)
- net D4: no longer U3.7 (UART_RX)
- net D5: no longer J3.2 (G2)
- net D8: no longer J14.2 (G2)
- net RADIO_RESET: now also J3.1 (G1)
- net at D1.1 (K), D2.1 (K), R12.2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: now also JP1.1; no longer C4.1, C5.1, U5.3 (VIN)
- net MISO renamed D12/MISO
- net D12/MISO: now also J3.2 (G2)
- net MOSI renamed D11/MOSI
- net D11/MOSI: now also U3.6 (UART_TX), J6.2 (G2)
- net SCK renamed D13/SCK
- new net: C4.1, C5.1, JP1.2, U5.3 (VIN)
- no-connect marks 40 -> 39
Other:
- note added: "Power LED TX ( red )"
- note added: "User LED RX ( green )"
- note removed: "User LED RX ( red )"
- moved on the sheet: C4, C5, C6, D5, J14, J3, P1, R14, U5

Commit message: near v0.7 ( mother and ext02 ), add mini extension
Parts:
- added JP2: Jumper_NC_Dual, Pin_Headers:Pin_Header_Straight_1x03_Pitch2.54mm, symbol Jumper_NC_Dual
- SW1: footprint w_switch:smd_push2 -> Buttons_Switches_THT:SW_Tactile_SPST_Angled_PTS645Vx58-2LFS
Connections:
- net D12/MISO: no longer J3.2 (G2)
- net D2: now also J6.1 (G1)
- net D3: now also JP2.1; no longer J6.1 (G1)
- net D9: now also J3.2 (G2)
- net RST: now also JP2.3; no longer SW1.2
- new net: JP2.2, SW1.2
Other:
- note added: "A0 =\nA1 =\nA2 = ATSHA204\nA3 = Battery Report\nA4 = SDA\nA5 = SCL\nA6 = RN2483 Rx LED \nA7 = RN2483 Tx LED\nD0 = RX\nD1 = TX\nD2 = ResetInterrupt ( from RN2483 ) or RFM69 DI0\nD3 = ButtonInterrupt ( ask for config )\nD4 =\nD5 =\nD6 =\nD7 = \nD8 =\nD9 = RN2483 Reset - RFM69 Reset\nD10 =RN2483 Rx - RFM69 NSS\nD11 = RN2483 Tx - RFM69 MOSI\nD12 = RFM69 MISO\nD13 = RFM69 SCK"
- note removed: "CONNECTORS"
- moved on the sheet: SW1
Changed lines of the file:
@@
 	1    0    0    -1
 $EndComp
-Text Notes 15250 2900 0    60   ~ 0
-CONNECTORS
 $Comp
 L SW_DIP_x01 SW1
 U 1 1 5978A193
-P 4050 3050
-F 0 "SW1" H 4050 3200 50  0000 C CNN
-F 1 "SW_DIP_x01" H 4050 2900 50  0000 C CNN
-F 2 "w_switch:smd_push2" H 4050 3050 50  0001 C CNN
-F 3 "" H 4050 3050 50  0001 C CNN
-	1    4050 3050
+P 4350 3300
+F 0 "SW1" H 4350 3450 50  0000 C CNN
+F 1 "SW_DIP_x01" H 4350 3150 50  0000 C CNN
+F 2 "Buttons_Switches_THT:SW_Tactile_SPST_Angled_PTS645Vx58-2LFS" H 4350 3300 50  0001 C CNN
+F 3 "" H 4350 3300 50  0001 C CNN
+	1    4350 3300
 	0    -1   -1   0
 $EndComp
@@
 L GND #PWR09
 U 1 1 597F4ED2
-P 4050 3450
-F 0 "#PWR09" H 4050 3200 50  0001 C CNN
-F 1 "GND" H 4050 3300 50  0000 C CNN
-F 2 "" H 4050 3450 50  0001 C CNN
-F 3 "" H 4050 3450 50  0001 C CNN
-	1    4050 3450
-	0    -1   -1   0
+P 4350 3600
+F 0 "#PWR09" H 4350 3350 50  0001 C CNN
+F 1 "GND" H 4350 3450 50  0000 C CNN
+F 2 "" H 4350 3600 50  0001 C CNN
+F 3 "" H 4350 3600 50  0001 C CNN
+	1    4350 3600
+	1    0    0    -1
 $EndComp
 $Comp
@@
 $EndComp
 Text GLabel 1500 5850 0    51   BiDi ~ 0
-D12/MISO
+D9
 Text Notes 7250 6450 0    47   ~ 0
 Charger Regulation - R11\n10K = 100mA\n5K = 200mA\n2K = 500mA\n1K = 1000mA
@@
 ANT
 Text GLabel 5150 7000 2    51   BiDi ~ 0
-D3
+D2
 Wire Wire Line
 	1050 1150 1600 1150
@@
 Wire Notes Line
 	7200 500  7200 6500
-Wire Wire Line
-	4050 3350 4050 3450
 Wire Wire Line
 	6200 4900 6600 4900
@@
 Wire Wire Line
 	8350 4650 8350 4750
+Text GLabel 4050 3250 3    51   BiDi ~ 0
+D3
+$Comp
+L Jumper_NC_Dual JP2
+U 1 1 5A2EFA3D
+P 4050 3000
+F 0 "JP2" H 4100 2900 50  0000 L CNN
+F 1 "Jumper_NC_Dual" H 4050 3100 50  0000 C BNN
+F 2 "Pin_Headers:Pin_Header_Straight_1x03_Pitch2.54mm" H 4050 3000 50  0001 C CNN
+F 3 "" H 4050 3000 50  0001 C CNN
+	1    4050 3000
+	0    -1   -1   0
+$EndComp
+Text Notes 550  7400 0    47   ~ 0
+A0 =\nA1 =\nA2 = ATSHA204\nA3 = Battery Report\nA4 = SDA\nA5 = SCL\nA6 = RN2483 Rx LED \nA7 = RN2483 Tx LED\nD0 = RX\nD1 = TX\nD2 = ResetInterrupt ( from RN2483 ) or RFM69 DI0\nD3 = ButtonInterrupt ( ask for config )\nD4 =\nD5 =\nD6 =\nD7 = \nD8 =\nD9 = RN2483 Reset - RFM69 Reset\nD10 =RN2483 Rx - RFM69 NSS\nD11 = RN2483 Tx - RFM69 MOSI\nD12 = RFM69 MISO\nD13 = RFM69 SCK
+Wire Wire Line
+	4150 3000 4350 3000
 $EndSCHEMATC
